Commit message: add again

File: rosws/src/myurdf/urdf/myurdf.urdf (robot description, URDF)
Before this commit: robot myurdf, 3 links, 2 joints
Links:
- added link back_left_steering, mass 0.610591222034383; collision mesh filename=package://myurdf/meshes/back_left_steering.STL; visual mesh filename=package://myurdf/meshes/back_left_steering.STL
- added link back_left_wheel, mass 0.265552463932757; collision mesh filename=package://myurdf/meshes/back_left_wheel.STL; visual mesh filename=package://myurdf/meshes/back_left_wheel.STL
- added link back_right_steering, mass 0.610591222475197; collision mesh filename=package://myurdf/meshes/back_right_steering.STL; visual mesh filename=package://myurdf/meshes/back_right_steering.STL
- added link back_right_wheel, mass 0.265552463932757; collision mesh filename=package://myurdf/meshes/back_right_wheel.STL; visual mesh filename=package://myurdf/meshes/back_right_wheel.STL
- added link front_left_steering, mass 0.61059122245919; collision mesh filename=package://myurdf/meshes/front_left_steering.STL; visual mesh filename=package://myurdf/meshes/front_left_steering.STL
- added link front_left_wheel, mass 0.265552463932756; collision mesh filename=package://myurdf/meshes/front_left_wheel.STL; visual mesh filename=package://myurdf/meshes/front_left_wheel.STL
- link base_link: mass 0.84428 -> 1.95577438158697
- link front_right_steering: mass 0.16386 -> 0.610591222095894
- link front_right_wheel: mass 0.22141 -> 0.265552463932757
Joints:
- added joint back_left_steering_joint: type continuous, parent base_link, child back_left_steering, origin xyz=0.23569 0.21808 0.033825 rpy=1.5708 0 1.0349, axis 0 -1 0
- added joint back_left_wheel_joint: type continuous, parent back_left_steering, child back_left_wheel, origin xyz=-0.0087483 -0.041 -0.0021067 rpy=-2.9038 -0.11023 -1.5975, axis 0 1 0
- added joint back_right_steering_joint: type continuous, parent base_link, child back_right_steering, origin xyz=-0.23631 0.21808 0.018015 rpy=1.5708 0 1.2169, axis 0 -1 0
- added joint back_right_wheel_joint: type continuous, parent back_right_steering, child back_right_wheel, origin xyz=0 -0.041 0 rpy=-2.9038 0 -1.5975, axis 0 1 0
- added joint front_left_steering_joint: type continuous, parent base_link, child front_left_steering, origin xyz=0.24069 -0.21508 0.030825 rpy=1.5708 0 -1.9247, axis 0 -1 0
- added joint front_left_wheel_joint: type continuous, parent front_left_steering, child front_left_wheel, origin xyz=-0.02147 -0.040515 -0.0048072 rpy=-2.753 -0.90465 -1.8822, axis 0 1 0
- joint front_right_steering_joint: origin xyz=0.083907 -0.21014 -0.02519 rpy=1.5708 0 -2.343 -> xyz=-0.23631 -0.21508 0.033825 rpy=1.5708 0 -2.1067
- joint front_right_wheel_joint: axis 0 0 1 -> 0 1 0; origin xyz=0.089441 0.017567 -0.0053214 rpy=1.5708 -1.1791 1.5708 -> xyz=-0.0087483 -0.041 -0.0021067 rpy=-2.9038 -0.11023 -1.5975
